Commit message: fix: correcion model_01

File: sauronbot_description/urdf/sauronbot.urdf.xacro (robot description, xacro)
@@ -97,7 +97,7 @@
   <link name="base_scan">
     <visual>
-      <origin xyz="0 -0.047 -0.031" rpy="0 0 0"/>
+      <origin xyz="0 0 0" rpy="0 0 0"/>
       <geometry>
-        <mesh filename="package://sauronbot_description/meshes/sensors/RPLIDAR_A3.stl" scale="0.001 0.001 0.001"/>
+        <mesh filename="package://sauronbot_description/meshes/sensors/RPLIDAR_A3_C.stl" scale="0.001 0.001 0.001"/>
       </geometry>
       <material name="light_black"/>

File: sauronbot_description/urdf/sauronbot_01.urdf.xacro (robot description, xacro)
@@ -14,7 +14,7 @@
   <link name="base_link">
     <visual>
-      <origin xyz="0.247 -0.125 -0.01723" rpy="1.57 0 3.14"/>
+      <origin xyz="0 0 0" rpy="0 0 0"/>
       <geometry>
-        <mesh filename="package://sauronbot_description/meshes/bases/sauronbot_base.stl" scale="0.001 0.001 0.001"/>
+        <mesh filename="package://sauronbot_description/meshes/bases/sauronbot_base_c.stl" scale="0.001 0.001 0.001"/>
       </geometry>
       <material name="light_black"/>
@@ -42,7 +42,7 @@
   <link name="wheel_left_link">
     <visual>
-      <origin xyz="-0.036 0 -0.01325" rpy="0 0 0"/>
+      <origin xyz="0 0 -0" rpy="0 0 0"/>
       <geometry>
-        <mesh filename="package://sauronbot_description/meshes/wheels/left_tire.stl" scale="0.001 0.001 0.001"/>
+        <mesh filename="package://sauronbot_description/meshes/wheels/left_tire_c.stl" scale="0.001 0.001 0.001"/>
       </geometry>
       <material name="dark"/>
@@ -72,5 +72,5 @@
       <origin xyz="0 0 0" rpy="0 0 0"/>
       <geometry>
-        <mesh filename="package://sauronbot_description/meshes/wheels/right_tire.stl" scale="0.001 0.001 0.001"/>
+        <mesh filename="package://sauronbot_description/meshes/wheels/right_tire_c.stl" scale="0.001 0.001 0.001"/>
       </geometry>
       <material name="dark"/>
@@ -93,11 +93,11 @@
     <parent link="base_link"/>
     <child link="base_scan"/>
-    <origin xyz="0.023 0 0.2144" rpy="0 0 0"/>
+    <origin xyz="-0.023 0 0.2144" rpy="0 0 0"/>
   </joint>
   <link name="base_scan">
     <visual>
-      <origin xyz="0 -0.047 -0.031" rpy="0 0 0"/>
+      <origin xyz="0 -0 0" rpy="0 0 0"/>
       <geometry>
-        <mesh filename="package://sauronbot_description/meshes/sensors/RPLIDAR_A3.stl" scale="0.001 0.001 0.001"/>
+        <mesh filename="package://sauronbot_description/meshes/sensors/RPLIDAR_A3_C.stl" scale="0.001 0.001 0.001"/>
       </geometry>
       <material name="light_black"/>
