Commit message: feat: add model_03

File: sauronbot_description/urdf/common_properties.xacro (robot description, xacro)
@@ -32,3 +32,6 @@
     <color rgba="1.0 1.0 1.0 1.0"/>
   </material>
+  <material name="RPICAMERA_V2_mat">
+        <color rgba="0.25 0.25 0.25 0.99"/>
+    </material>
 </robot>
