Commit message: feat: model3: realsense d435

File: sauronbot_description/urdf/sauronbot_model_03.urdf.xacro (robot description, xacro)
@@ -12,4 +12,13 @@
   <xacro:arg name="cam_pitch"     default="0.0" />
   <xacro:arg name="cam_yaw"       default="0.0" />
+  <xacro:arg name="depth_camera_name"   default="realsese_d435" />
+  <xacro:arg name="depth_camera_model"  default="SOPORTE_REALSENSE_D435" />
+  <xacro:arg name="depth_base_frame"    default="base_link" />
+  <xacro:arg name="depth_cam_pos_x"     default="-0.08149" />
+  <xacro:arg name="depth_cam_pos_y"     default="0.0" />
+  <xacro:arg name="depth_cam_pos_z"     default="0.345" />
+  <xacro:arg name="depth_cam_roll"      default="0.0" />
+  <xacro:arg name="depth_cam_pitch"     default="0.0" />
+  <xacro:arg name="depth_cam_yaw"       default="0.0" />
   <!-- Properties -->
 	<xacro:property name="r200_cam_rgb_px" value="0.005"/>
@@ -17,5 +26,6 @@
   <xacro:property name="r200_cam_rgb_pz" value="0.013"/>
   <xacro:property name="r200_cam_depth_offset" value="0.01"/>
-  <xacro:property name="camera_model_stl"    value="$(arg camera_model)" />
+  <xacro:property name="camera_model_stl"           value="$(arg camera_model)" />
+  <xacro:property name="depth_camera_model_stl"     value="$(arg depth_camera_model)" />
   <link name="base_footprint"/>
   <joint name="base_joint" type="fixed">
@@ -162,3 +172,29 @@
   </joint>
   <link name="$(arg camera_name)_camera_rgb_optical_frame"/>
+  <!-- Depth Camara -->
+  <joint name="$(arg depth_camera_name)_camera_joint" type="fixed">
+    <origin xyz="$(arg depth_cam_pos_x) $(arg depth_cam_pos_y) $(arg depth_cam_pos_z)" rpy="$(arg depth_cam_roll) $(arg depth_cam_pitch) $(arg depth_cam_yaw)"/>
+    <parent link="$(arg depth_base_frame)"/>
+    <child link="$(arg depth_camera_name)_base_link"/>
+  </joint>
+  <xacro:arg name="use_nominal_extrinsics" default="false"/>
+  <xacro:include filename="$(find sauronbot_description)/urdf/_d435.urdf.xacro" />
+  <link name="$(arg depth_camera_name)_base_link">
+    <collision>
+      <origin xyz="0 0 0" rpy="0 0 0"/>
+      <geometry>
+        <box size="0.015 0.030 0.027"/>
+      </geometry>
+    </collision>
+    <visual>
+      <origin xyz="0 0 0" rpy="0 0 0"/>
+      <geometry>
+        <mesh filename="package://sauronbot_description/meshes/sensors/${depth_camera_model_stl}.STL" scale="0.001 0.001 0.001"/>
+      </geometry>
+      <material name="${camera_model_stl}_mat" />
+    </visual>
+  </link>
+  <xacro:sensor_d435 parent="$(arg depth_camera_name)_base_link" use_nominal_extrinsics="$(arg use_nominal_extrinsics)">
+    <origin xyz="0 0 0.01201" rpy="0 0 0"/>
+  </xacro:sensor_d435>
 </robot>

Commit message: feat: add model for gazebo

File: sauronbot_description/urdf/sauronbot_model_03.urdf.xacro (robot description, xacro)
@@ -21,4 +21,5 @@
   <xacro:arg name="depth_cam_pitch"     default="0.0" />
   <xacro:arg name="depth_cam_yaw"       default="0.0" />
+  <xacro:include filename="$(find sauronbot_description)/urdf/include/sauronbot_model_03.gazebo.xacro"/>
   <!-- Properties -->
 	<xacro:property name="r200_cam_rgb_px" value="0.005"/>
@@ -38,4 +39,5 @@
       <origin xyz="0 0 0" rpy="0 0 0"/>
       <geometry>
+        <!-- <mesh filename="package://sauronbot_description/meshes/bases/BASE_MODEL_03_-.STL" scale="0.001 0.001 0.001"/> -->
         <mesh filename="package://sauronbot_description/meshes/bases/BASE_MODEL_03.STL" scale="0.001 0.001 0.001"/>
       </geometry>
@@ -45,5 +47,6 @@
       <origin xyz="0 0 0" rpy="0 0 0"/>
       <geometry>
-        <box size="0.266 0.266 0.094"/>
+        <!-- <box size="0.266 0.266 0.094"/> -->
+        <mesh filename="package://sauronbot_description/meshes/bases/BASE_MODEL_03.STL" scale="0.001 0.001 0.001"/>
       </geometry>
     </collision>
@@ -73,5 +76,6 @@
       <origin xyz="0 0 0" rpy="0 0 0"/>
       <geometry>
-        <cylinder length="0.018" radius="0.033"/>
+        <!-- <cylinder length="0.018" radius="0.033"/> -->
+        <mesh filename="package://sauronbot_description/meshes/wheels/WHEEL_LEFT.STL" scale="0.001 0.001 0.001"/>
       </geometry>
     </collision>
@@ -101,5 +105,6 @@
       <origin xyz="0 0 0" rpy="0 0 0"/>
       <geometry>
-        <cylinder length="0.018" radius="0.033"/>
+        <!-- <cylinder length="0.018" radius="0.033"/> -->
+        <mesh filename="package://sauronbot_description/meshes/wheels/WHEEL_RIGHT.STL" scale="0.001 0.001 0.001"/>
       </geometry>
     </collision>

Commit message: fix: correccion D435

File: sauronbot_description/urdf/sauronbot_model_03.urdf.xacro (robot description, xacro)
@@ -6,5 +6,5 @@
   <xacro:arg name="camera_model"  default="RPICAMERA_V2" />
   <xacro:arg name="base_frame"    default="base_link" />
-  <xacro:arg name="cam_pos_x"     default="0.07089" />
+  <xacro:arg name="cam_pos_x"     default="0.07989" />
   <xacro:arg name="cam_pos_y"     default="0.0" />
   <xacro:arg name="cam_pos_z"     default="0.0801" />
@@ -40,5 +40,5 @@
       <geometry>
         <!-- <mesh filename="package://sauronbot_description/meshes/bases/BASE_MODEL_03_-.STL" scale="0.001 0.001 0.001"/> -->
-        <mesh filename="package://sauronbot_description/meshes/bases/BASE_MODEL_03.STL" scale="0.001 0.001 0.001"/>
+        <mesh filename="package://sauronbot_description/meshes/bases/BASE_MODEL_03_-.STL" scale="0.001 0.001 0.001"/>
       </geometry>
       <material name="light_black"/>
@@ -53,5 +53,5 @@
     <inertial>
       <origin xyz="0 0 0" rpy="0 0 0"/>
-      <mass value="1.3729096e+00"/>
+      <mass value="3.57516e+00"/>
       <inertia ixx="8.7002718e-03" ixy="-4.7576583e-05" ixz="1.1160499e-04"
                iyy="8.6195418e-03" iyz="-3.5422299e-06"
@@ -199,7 +199,14 @@
       <material name="${camera_model_stl}_mat" />
     </visual>
+<!--     <inertial>
+      <origin xyz="0 0 0" rpy="0 0 0"/>
+      <mass value="1.3729096e+00"/>
+      <inertia ixx="8.7002718e-03" ixy="-4.7576583e-05" ixz="1.1160499e-04"
+               iyy="8.6195418e-03" iyz="-3.5422299e-06"
+               izz="1.4612727e-02" />
+    </inertial> -->
   </link>
   <xacro:sensor_d435 parent="$(arg depth_camera_name)_base_link" use_nominal_extrinsics="$(arg use_nominal_extrinsics)">
-    <origin xyz="0 0 0.01201" rpy="0 0 0"/>
+    <origin xyz="0.00015 0 0.011" rpy="0 0 0"/>
   </xacro:sensor_d435>
 </robot>

Commit message: feat: add inercia: base_link, realsenseD435_base_link

File: sauronbot_description/urdf/sauronbot_model_03.urdf.xacro (robot description, xacro)
@@ -52,9 +52,9 @@
     </collision>
     <inertial>
-      <origin xyz="0 0 0" rpy="0 0 0"/>
-      <mass value="3.57516e+00"/>
-      <inertia ixx="8.7002718e-03" ixy="-4.7576583e-05" ixz="1.1160499e-04"
-               iyy="8.6195418e-03" iyz="-3.5422299e-06"
-               izz="1.4612727e-02" />
+      <origin xyz="-0.07724994 0.00010247 0.07636139" rpy="0 0 0"/>
+      <mass value="3.57515504e+00"/>
+      <inertia ixx="47.13236e-03" ixy="88.68e-09" ixz="-24.5273e-04"
+               iyy="46.11917e-03" iyz="-9.0e-06"
+               izz="7.414357e-02" />
     </inertial>
   </link>
@@ -199,11 +199,11 @@
       <material name="${camera_model_stl}_mat" />
     </visual>
-<!--     <inertial>
-      <origin xyz="0 0 0" rpy="0 0 0"/>
-      <mass value="1.3729096e+00"/>
-      <inertia ixx="8.7002718e-03" ixy="-4.7576583e-05" ixz="1.1160499e-04"
-               iyy="8.6195418e-03" iyz="-3.5422299e-06"
-               izz="1.4612727e-02" />
-    </inertial> -->
+     <inertial>
+      <origin xyz="-0.08176576 -0.00005103 0.24947569" rpy="0 0 0"/>
+      <mass value="0.05701498e+00"/>
+      <inertia ixx="0.24961e-03" ixy="20e-09" ixz="-1.05e-06"
+               iyy="0.24976e-03" iyz="-0.25e-06"
+               izz="10.363268e-06" />
+    </inertial>
   </link>
   <xacro:sensor_d435 parent="$(arg depth_camera_name)_base_link" use_nominal_extrinsics="$(arg use_nominal_extrinsics)">

Commit message: feat: correcion model_03

File: sauronbot_description/urdf/sauronbot_model_03.urdf.xacro (robot description, xacro)
@@ -40,5 +40,5 @@
       <geometry>
         <!-- <mesh filename="package://sauronbot_description/meshes/bases/BASE_MODEL_03_-.STL" scale="0.001 0.001 0.001"/> -->
-        <mesh filename="package://sauronbot_description/meshes/bases/BASE_MODEL_03_-.STL" scale="0.001 0.001 0.001"/>
+        <mesh filename="package://sauronbot_description/meshes/bases/BASE_MODEL_03.STL" scale="0.001 0.001 0.001"/>
       </geometry>
       <material name="light_black"/>
